File: kicad/kicad.kicad_pcb (KiCad board)
At the start: 2 copper layers, 307 x 30 mm, 18 parts

Commit message: Add files
Parts:
- removed the G*** at (101.5, 111.0)
- added G***: LOGO, personal:qrcode, B.Cu at (290.0, 109.8)
- added REF**: TSSOP-8_4.4x3mm_P0.65mm, Package_SO:TSSOP-8_4.4x3mm_P0.65mm, B.Cu at (40.0, 101.0)
- added REF**: TO-263-2, Package_TO_SOT_SMD:TO-263-2, B.Cu at (149.0, 102.0)
- added REF**: KiCad-Logo2_5mm_SilkScreen, Symbol:KiCad-Logo2_5mm_SilkScreen, B.Cu at (321.0, 115.5)
- added REF**: Symbol_CreativeCommons_CopperTop_Type2_Small, personal:Symbol_CreativeCommons_SilkTop_Type2_Small, B.Cu at (332.0, 115.5)
- added REF**: D_SOD-923, Diode_SMD:D_SOD-923, B.Cu at (75.8, 117.0)
- added REF**: D_SOD-523, Diode_SMD:D_SOD-523, B.Cu at (75.8, 112.0)
- added REF**: D_SOD-323, Diode_SMD:D_SOD-323, B.Cu at (75.8, 106.0)
- added REF**: D_SOD-123, Diode_SMD:D_SOD-123, B.Cu at (76.0, 100.0)
- added REF**: D_SMA, Diode_SMD:D_SMA, B.Cu at (87.0, 117.0)
- added REF**: D_SMB, Diode_SMD:D_SMB, B.Cu at (87.0, 109.0)
- added REF**: D_SMC, Diode_SMD:D_SMC, B.Cu at (87.0, 100.0)
- added REF**: VSSOP-10_3x3mm_P0.5mm, Package_SO:VSSOP-10_3x3mm_P0.5mm, B.Cu at (40.0, 113.0)
- added REF**: SW_Push_1P1T_NO_CK_KMR2, Button_Switch_SMD:SW_Push_1P1T_NO_CK_KMR2, B.Cu at (109.0, 115.0)
- added REF**: SW_DPDT_CK_JS202011JCQN, Button_Switch_SMD:SW_DPDT_CK_JS202011JCQN, B.Cu at (109.0, 103.0)
- added REF**: D_2512_6332Metric, Diode_SMD:D_2512_6332Metric, B.Cu at (169.8, 107.0)
- added REF**: D_2010_5025Metric, Diode_SMD:D_2010_5025Metric, B.Cu at (174.0, 107.0)
- added REF**: C_1210_3225Metric, Capacitor_SMD:C_1210_3225Metric, B.Cu at (178.0, 107.0)
- added REF**: C_1206_3216Metric, Capacitor_SMD:C_1206_3216Metric, B.Cu at (181.5, 107.0)
- added REF**: C_0805_2012Metric, Capacitor_SMD:C_0805_2012Metric, B.Cu at (184.5, 107.0)
- added REF**: C_0603_1608Metric, Capacitor_SMD:C_0603_1608Metric, B.Cu at (187.0, 107.0)
- added REF**: C_0402_1005Metric, Capacitor_SMD:C_0402_1005Metric, B.Cu at (189.5, 107.0)
- added REF**: C_0201_0603Metric, Capacitor_SMD:C_0201_0603Metric, B.Cu at (191.5, 107.0)
- added REF**: LQFP-64_7x7mm_P0.4mm, Package_QFP:LQFP-64_7x7mm_P0.4mm, B.Cu at (52.0, 113.0)
- added REF**: L_12x12mm_H8mm, Inductor_SMD:L_12x12mm_H8mm, B.Cu at (230.5, 102.5)
- added REF**: L_10.4x10.4_H4.8, Inductor_SMD:L_10.4x10.4_H4.8, B.Cu at (214.5, 102.8)
- added REF**: L_7.3x7.3_H4.5, Inductor_SMD:L_7.3x7.3_H4.5, B.Cu at (230.2, 114.5)
- added REF**: L_6.3x6.3_H3, Inductor_SMD:L_6.3x6.3_H3, B.Cu at (214.2, 114.2)
- added REF**: inch_ruler_10, personal:inch_ruler_10, B.Cu at (31.0, 90.0)
- added REF**: LQFP-36_7x7mm_P0.65mm, Package_QFP:LQFP-36_7x7mm_P0.65mm, B.Cu at (52.0, 101.0)
- added REF**: SOT-23, Package_TO_SOT_SMD:SOT-23, B.Cu at (142.0, 114.0)
- added REF**: SOT-223, Package_TO_SOT_SMD:SOT-223, B.Cu at (152.0, 114.0)
- added REF**: SOT-563, Package_TO_SOT_SMD:SOT-563, B.Cu at (128.0, 114.0)
- added REF**: SOT-363_SC-70-6, Package_TO_SOT_SMD:SOT-363_SC-70-6, B.Cu at (135.0, 114.0)
- added REF**: TO-252-2, Package_TO_SOT_SMD:TO-252-2, B.Cu at (131.0, 102.0)
- moved G*** 10.5 mm to (102.0, 111.0)
- moved E$53 6.50 mm to (112.5, 111.5)
- moved REF** 2.50 mm to (47.5, 103.5)
Routing:
- net (no net): track 0.00 -> 129.4 mm
Other:
- board text added: "+10/50°C"
- board text added: "0.6A/1.2A"
- board text added: "0.8A/1.5A"
- board text added: "0.9A/1.8A"
- board text added: "0201"
- board text added: "0402"
- board text added: "0603"
- board text added: "0805"
- board text added: "1"
- board text added: "1.0A/2.0A"
- board text added: "1.1A/2.3A"
- board text added: "1.2A/2.5A"
- board text added: "1.4A/2.8A"
- board text added: "1.5A/3.0A"
- board text added: "1.7A/3.4A"
- board text added: "1.9A/3.8A"
- board text added: "1/10"
- board text added: "1/16"
- board text added: "1/2"
- board text added: "1/20"
- board text added: "1/4"
- board text added: "1/8"
- board text added: "10.4x10.4"
- board text added: "10/0.25"
- board text added: "12/0.30"
- board text added: "1206"
- board text added: "1210"
- board text added: "12x12"
- board text added: "14/0.35"
- board text added: "16/0.40"
- board text added: "18/0.45"
- board text added: "2.0A/4.0A"
- board text added: "2.1A/4.1A"
- board text added: "2.4A/4.9A"
- board text added: "20/0.50"
- board text added: "2010"
- board text added: "24/0.60"
- board text added: "2512"
- board text added: "28/0.70"
- board text added: "3/4"
- board text added: "30/0.76"
- board text added: "32/0.80"
- board text added: "35µm=1.4mil"
- board text added: "40/1.00"
- board text added: "6.3x6.3"
- board text added: "6/0.15"
- board text added: "7.3x7.3"
- board text added: "8/0.20"
- board text added: "Diodes"
- board text added: "E12: 1.0, 1.2, 1.5, 1.8, 2.2, 2.7, 3.3, 3.9, 4.7, 5.6, 6.8, 8.2"
- board text added: "EIA (in)"
- board text added: "Inductors"
- board text added: "JLCJLCJLCJLC"
- board text added: "JS202011SCQN"
- board text added: "KMR2"
- board text added: "Misc."
- board text added: "Pow. (W)"
- board text added: "QFP-36"
- board text added: "QFP-64"
- board text added: "RLC"
- board text added: "SMA"
- board text added: "SMB"
- board text added: "SMC"
- board text added: "SOD123"
- board text added: "SOD323"
- board text added: "SOD523"
- board text added: "SOD923"
- board text added: "SOT-223"
- board text added: "SOT-23"
- board text added: "SOT-363"
- board text added: "SOT-563"
- board text added: "Switches"
- board text added: "TO-252"
- board text added: "TO-263"
- board text added: "TSSOP-8"
- board text added: "Transistors"
- board text added: "UIUC PCB Ruler v1 2021/09/06 Nebhrajani A. V."
- board text added: "VSSOP-10"
- board text added: "mil/mm"
- board text added: "www.illinois.edu"
